Commit message: questions on base_footprint, frames, and inertia

File: my_rb1_description/urdf/my_rb1_robot.urdf (robot description, URDF)
Before this commit: robot None, 0 links, 0 joints
Links:
- added link , mass 0; collision cylinder length= radius=; visual cylinder length= radius=

Commit message: inertia tensors added for links

File: my_rb1_description/urdf/my_rb1_robot.urdf (robot description, URDF)
Before this commit: robot my_rb1_robot, 1 links, 0 joints
Links:
- removed link 
- added link base_footprint; visual cylinder length=0.001 radius=0.25
- added link base_link, mass 24.926; collision cylinder length=0.3 radius=0.25; visual cylinder length=0.3 radius=0.25
- added link front_caster, mass 0.006; collision sphere radius=0.015; collision sphere radius=0.025
- added link front_laser, mass 0.021; collision cylinder length=0.025 radius=0.025; visual cylinder length=0.025 radius=0.025
- added link left_wheel, mass 0.021; collision cylinder length=0.025 radius=0.025; visual cylinder length=0.025 radius=0.025
- added link rear_caster, mass 0.006; collision sphere radius=0.015; collision sphere radius=0.025
- added link right_wheel, mass 0.021; collision cylinder length=0.025 radius=0.025; visual cylinder length=0.025 radius=0.025
Joints:
- added joint joint_base_footprint_base_link: type fixed, parent base_footprint, child base_link, origin xyz=0 0 0.15 rpy=0 0 0
- added joint joint_base_link_front_caster: type fixed, parent base_link, child front_caster, origin xyz=0.1 0.0 -0.15 rpy=0 0 0
- added joint joint_base_link_front_laser: type fixed, parent base_link, child front_laser, origin xyz=0.25 0.0 0.075 rpy=3.14159 0 0
- added joint joint_base_link_left_wheel: type continuous, parent base_link, child left_wheel, origin xyz=0 0.2 -0.15 rpy=1.5708 0 0, axis 0 0 1, limit effort=1000 velocity=1000
- added joint joint_base_link_rear_caster: type fixed, parent base_link, child rear_caster, origin xyz=-0.1 0.0 -0.15 rpy=0 0 0
- added joint joint_base_link_right_wheel: type continuous, parent base_link, child right_wheel, origin xyz=0 -0.2 -0.15 rpy=1.5708 0 0, axis 0 0 1, limit effort=1000 velocity=1000

Commit message: experimenting with friction coefficients

File: my_rb1_description/urdf/my_rb1_robot.urdf (robot description, URDF)
Before this commit: robot experiment, 7 links, 6 joints
Joints:
- joint joint_base_link_left_wheel: limit effort=1000 velocity=1000 -> effort=10000 velocity=1000
- joint joint_base_link_right_wheel: limit effort=1000 velocity=1000 -> effort=10000 velocity=1000
