Commit message: experimenting with links and joints

File: my_rb1_description/urdf/experiment.urdf (robot description, URDF)
Before this commit: robot my_rb1_robot, 1 links, 0 joints
Links:
- removed link 
- added link base_link, mass 0; collision cylinder length=0.3 radius=0.25; visual cylinder length=0.3 radius=0.25

Commit message: exp footprint joint base

File: my_rb1_description/urdf/experiment.urdf (robot description, URDF)
Before this commit: robot experiment, 1 links, 0 joints
Links:
- added link base_footprint; visual cylinder length=0.001 radius=0.25
- link base_link: mass 0 -> None
Joints:
- added joint joint_base_footprint_base_link: type fixed, parent base_footprint, child base_link, origin xyz=0 0 0.301 rpy=0 0 0

Commit message: all links, no mass, no inert

File: my_rb1_description/urdf/experiment.urdf (robot description, URDF)
Before this commit: robot experiment, 2 links, 1 joints
Links:
- added link front_caster; collision sphere radius=0.015; collision sphere radius=0.025
- added link front_laser; collision cylinder length=0.025 radius=0.025; visual cylinder length=0.025 radius=0.025
- added link left_wheel; collision cylinder length=0.025 radius=0.025; visual cylinder length=0.025 radius=0.025
- added link rear_caster; collision sphere radius=0.015; collision sphere radius=0.025
- added link right_wheel; collision cylinder length=0.025 radius=0.025; visual cylinder length=0.025 radius=0.025
Joints:
- added joint joint_base_link_front_caster: type fixed, parent base_link, child front_caster, origin xyz=0.1 0.0 -0.15 rpy=0 0 0
- added joint joint_base_link_front_laser: type fixed, parent base_link, child front_laser, origin xyz=0.25 0.0 0.075 rpy=3.14159 0 0
- added joint joint_base_link_left_wheel: type continuous, parent base_link, child left_wheel, origin xyz=0 0.2 -0.15 rpy=1.5708 0 0, axis 0 0 1, limit effort=1000 velocity=1000
- added joint joint_base_link_rear_caster: type fixed, parent base_link, child rear_caster, origin xyz=-0.1 0.0 -0.15 rpy=0 0 0
- added joint joint_base_link_right_wheel: type continuous, parent base_link, child right_wheel, origin xyz=0 -0.2 -0.15 rpy=1.5708 0 0, axis 0 0 1, limit effort=1000 velocity=1000
- joint joint_base_footprint_base_link: origin xyz=0 0 0.301 rpy=0 0 0 -> xyz=0 0 0.15 rpy=0 0 0

Commit message: added masses

File: my_rb1_description/urdf/experiment.urdf (robot description, URDF)
Before this commit: robot experiment, 7 links, 6 joints
Links:
- link base_link: mass None -> 24.926
- link front_caster: mass None -> 0.006
- link front_laser: mass None -> 0.021
- link left_wheel: mass None -> 0.021
- link rear_caster: mass None -> 0.006
- link right_wheel: mass None -> 0.021

Commit message: unwanted motion fixed, wront direction of motion

File: my_rb1_description/urdf/experiment.urdf (robot description, URDF)
Before this commit: robot my_rb1_robot, 7 links, 6 joints
Links:
- link base_link: mass 24.926 -> 22.5
- link front_caster: mass 0.006 -> 0.5
- link front_laser: mass 0.021 -> 0.5
- link left_wheel: mass 0.021 -> 0.5
- link rear_caster: mass 0.006 -> 0.5
- link right_wheel: mass 0.021 -> 0.5

Commit message: reverse fixed, task 3 completed

File: my_rb1_description/urdf/experiment.urdf (robot description, URDF)
Before this commit: robot my_rb1_robot, 7 links, 6 joints
Joints:
- joint joint_base_link_left_wheel: origin xyz=0 0.2 -0.15 rpy=1.5708 0 0 -> xyz=0 0.2 -0.15 rpy=1.5708 0 3.14159
- joint joint_base_link_right_wheel: origin xyz=0 -0.2 -0.15 rpy=1.5708 0 0 -> xyz=0 -0.2 -0.15 rpy=1.5708 0 3.14159

File: my_rb1_description/urdf/my_rb1_robot.urdf (robot description, URDF)
Before this commit: robot my_rb1_robot, 7 links, 6 joints
Links:
- link base_link: mass 24.926 -> 22.5
- link front_caster: mass 0.006 -> 0.5
- link front_laser: mass 0.021 -> 0.5
- link left_wheel: mass 0.021 -> 0.5
- link rear_caster: mass 0.006 -> 0.5
- link right_wheel: mass 0.021 -> 0.5
Joints:
- joint joint_base_link_left_wheel: origin xyz=0 0.2 -0.15 rpy=1.5708 0 0 -> xyz=0 0.2 -0.15 rpy=1.5708 0 3.14159
- joint joint_base_link_right_wheel: origin xyz=0 -0.2 -0.15 rpy=1.5708 0 0 -> xyz=0 -0.2 -0.15 rpy=1.5708 0 3.14159
